File: RC_Sounds.kicad_pcb (KiCad board)
At the start: 2 copper layers, 67.9 x 42.5 mm, 59 parts, among them J1 CONN_02, J2 REPROG, J3 CONN_03, J4 CONN_02, J5 CONN_04, J6 EXT AUDIO, J7 BEC ENABLE, M1 Motor_Servo_JR, M2 Motor_Servo_JR, SW1 SW_DIP_x04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

Commit message: Add files via upload
Corrected error in analogue input connection in schematic and PCB.
Parts:
- D1: value LED1 -> LED-GREEN0603
- J2: value REPROG -> AVR_SPI_PROG_3X2PTH
- J6: value EXT AUDIO -> CONN_04
- J7: value BEC ENABLE -> CONN_02
- S1: value SETUP -> MOMENTARY-SWITCH
- moved R6 23.7 mm to (192.8, 76.5), turned to 180 degrees
Connections:
- R10 pad 1: Net-(R10-Pad1) -> Net-(J2-Pad5)
- R11 pad 1: Net-(R10-Pad1) -> Net-(J2-Pad5)
- R12 pad 1: Net-(R10-Pad1) -> Net-(J2-Pad5)
- R13 pad 1: Net-(R10-Pad1) -> Net-(J2-Pad5)
- R6 pad 1: Net-(R10-Pad1) -> Net-(J2-Pad5)
- R8 pad 2: Net-(R10-Pad1) -> Net-(J2-Pad5)
- R9 pad 1: Net-(R10-Pad1) -> Net-(J2-Pad5)
Routing:
- net Net-(R6-Pad2): track 47.5 -> 7.97 mm
- net Net-(J2-Pad5): track 34.7 -> 64.6 mm
- net Net-(R10-Pad1): track 21.0 -> 0.00 mm
- net /RX_MICRO: track 11.5 -> 17.0 mm
- net GND: track 192.6 -> 190.5 mm
