File: RC_Sounds.sch (KiCad schematic (older format))
At the start: 59 parts, among them J1 CONN_02, J2 AVR_SPI_PROG_3X2PTH, J3 CONN_03, J4 CONN_02, J5 CONN_04, J6 CONN_04, J7 CONN_02, M1 Motor_Servo_JR, M2 Motor_Servo_JR, SW1 SW_DIP_x04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

Commit message: Add files via upload
Corrected error in analogue input connection in schematic and PCB.
Parts:
- D1: symbol SparkFun-LED:LED-GREEN0603 -> RC_Sounds-rescue:LED-GREEN0603-SparkFun-LED
- H1, H2, H3, H4: symbol SparkFun-Hardware:STAND-OFFTIGHT -> RC_Sounds-rescue:STAND-OFFTIGHT-SparkFun-Hardware
- J1, J7: symbol Sparkfun_connectors:CONN_02 -> RC_Sounds-rescue:CONN_02-Sparkfun_connectors
- J2: symbol Sparkfun_connectors:AVR_SPI_PROG_3X2PTH -> RC_Sounds-rescue:AVR_SPI_PROG_3X2PTH-Sparkfun_connectors
- J3: symbol SparkFun-Connectors:CONN_03 -> RC_Sounds-rescue:CONN_03-SparkFun-Connectors
- J4: symbol SparkFun-Connectors:CONN_02 -> RC_Sounds-rescue:CONN_02-SparkFun-Connectors
- J5, J6: symbol SparkFun-Connectors:CONN_04 -> RC_Sounds-rescue:CONN_04-SparkFun-Connectors
- R17: symbol PTV112:PTV112 -> RC_Sounds-rescue:PTV112-PTV112
- S1: symbol SparkFun-Switches:MOMENTARY-SWITCH-SPST-SMD-5.2MM -> RC_Sounds-rescue:MOMENTARY-SWITCH-SPST-SMD-5.2MM-SparkFun-Switches
- U2: symbol MCU_Microchip_ATtiny:ATtiny85-20SU -> RC_Sounds-rescue:ATtiny85-20SU-MCU_Microchip_ATtiny
- U3: symbol PAM8403DR:PAM8403DR -> RC_Sounds-rescue:PAM8403DR-PAM8403DR
- U4: symbol DFR0299:DFR0299 -> RC_Sounds-rescue:DFR0299-DFR0299
Connections:
- wire segments 265 -> 267
Other:
- note added: "Missing on V1.1 PCB\n"
Changed lines of the file:
@@
 $EndDescr
 $Comp
-L DFR0299:DFR0299 U4
+L RC_Sounds-rescue:DFR0299-DFR0299 U4
 U 1 1 5F908738
 P 8900 3100
@@
 $EndComp
 $Comp
-L PAM8403DR:PAM8403DR U3
+L RC_Sounds-rescue:PAM8403DR-PAM8403DR U3
 U 1 1 5F918A9D
 P 4750 8950
@@
 Connection ~ 5850 8450
 $Comp
-L Sparkfun_connectors:CONN_02 J1
+L RC_Sounds-rescue:CONN_02-Sparkfun_connectors J1
 U 1 1 5F97EFE6
 P 5250 10400
@@
 Connection ~ 7350 9300
 $Comp
-L Sparkfun_connectors:AVR_SPI_PROG_3X2PTH J2
+L RC_Sounds-rescue:AVR_SPI_PROG_3X2PTH-Sparkfun_connectors J2
 U 1 1 5FBC0777
 P 6300 2300
@@
 PB5 Analogue in/switch\nPB2 LED\nPB1 (horn)\nPB0 (Aux in for horn)
 $Comp
-L MCU_Microchip_ATtiny:ATtiny85-20SU U2
+L RC_Sounds-rescue:ATtiny85-20SU-MCU_Microchip_ATtiny U2
 U 1 1 5FA14CF5
 P 4500 3350
@@
 	6100 6500 6150 6500
 $Comp
-L SparkFun-Switches:MOMENTARY-SWITCH-SPST-SMD-5.2MM S1
+L RC_Sounds-rescue:MOMENTARY-SWITCH-SPST-SMD-5.2MM-SparkFun-Switches S1
 U 1 1 5FE2E806
 P 4950 5700
@@
 	4950 5900 4950 6100
 $Comp
-L SparkFun-Connectors:CONN_03 J3
+L RC_Sounds-rescue:CONN_03-SparkFun-Connectors J3
 U 1 1 5FE6A2C7
 P 7150 4000
@@
 	7850 1450 9650 1450
 $Comp
-L SparkFun-Connectors:CONN_04 J6
+L RC_Sounds-rescue:CONN_04-SparkFun-Connectors J6
 U 1 1 6001321B
 P 12500 2900
@@
 Connection ~ 12250 3100
 $Comp
-L SparkFun-Connectors:CONN_04 J5
+L RC_Sounds-rescue:CONN_04-SparkFun-Connectors J5
 U 1 1 60056A94
 P 10550 8900
@@
 	7350 9300 10350 9300
 $Comp
-L SparkFun-Connectors:CONN_02 J4
+L RC_Sounds-rescue:CONN_02-SparkFun-Connectors J4
 U 1 1 600ACA5E
 P 1400 1550
@@
 Optional speed/aux input
 $Comp
-L SparkFun-LED:LED-GREEN0603 D1
+L RC_Sounds-rescue:LED-GREEN0603-SparkFun-LED D1
 U 1 1 60137D2D
 P 7550 2050
@@
 	7050 2050 7350 2050
 $Comp
-L PTV112:PTV112 R17
+L RC_Sounds-rescue:PTV112-PTV112 R17
 U 1 1 60199D6D
 P 10350 3550
@@
 $EndComp
 $Comp
-L PTV112:PTV112 R17
+L RC_Sounds-rescue:PTV112-PTV112 R17
 U 2 1 6019E190
 P 10650 2800
@@
 	10650 2450 10650 2500
 $Comp
-L SparkFun-Hardware:STAND-OFFTIGHT H1
+L RC_Sounds-rescue:STAND-OFFTIGHT-SparkFun-Hardware H1
 U 1 1 602F0EFC
 P 15000 9000
@@
 $EndComp
 $Comp
-L SparkFun-Hardware:STAND-OFFTIGHT H2
+L RC_Sounds-rescue:STAND-OFFTIGHT-SparkFun-Hardware H2
 U 1 1 602F1C12
 P 15000 9150
@@
 $EndComp
 $Comp
-L SparkFun-Hardware:STAND-OFFTIGHT H3
+L RC_Sounds-rescue:STAND-OFFTIGHT-SparkFun-Hardware H3
 U 1 1 602F1E75
 P 15000 9300
@@
 $EndComp
 $Comp
-L SparkFun-Hardware:STAND-OFFTIGHT H4
+L RC_Sounds-rescue:STAND-OFFTIGHT-SparkFun-Hardware H4
 U 1 1 602F1FF8
 P 15000 9450
@@
 $EndComp
 $Comp
-L Sparkfun_connectors:CONN_02 J7
+L RC_Sounds-rescue:CONN_02-Sparkfun_connectors J7
 U 1 1 5FC3DC7E
 P 3900 1900
@@
 	7050 3550 7500 3550
 Wire Wire Line
-	5100 3550 5950 3550
+	5100 3550 5400 3550
 Wire Wire Line
 	5100 3150 5150 3150
@@
 	4950 4500 4950 5000
 Wire Wire Line
-	5400 2200 5400 4500
+	5400 2200 5400 3550
 Connection ~ 5400 4500
 Wire Wire Line
 	5400 4500 5400 4800
 $Comp
-L power:GND #PWR?
+L power:GND #PWR0102
 U 1 1 60A2B37A
 P 7600 4100
-F 0 "#PWR?" H 7600 3850 50  0001 C CNN
+F 0 "#PWR0102" H 7600 3850 50  0001 C CNN
 F 1 "GND" H 7605 3927 50  0000 C CNN
 F 2 "" H 7600 4100 50  0001 C CNN
@@
 Wire Wire Line
 	7500 3550 7700 3550
+Connection ~ 5400 3550
+Wire Wire Line
+	5400 3550 5950 3550
+Wire Wire Line
+	5400 3550 5400 4500
+Text Notes 5400 3650 0    50   ~ 0
+Missing on V1.1 PCB\n
 $EndSCHEMATC
